File: dimmer-board/dimmer-board.kicad_sch (KiCad schematic)
At the start: 16 parts, among them J1 Conn_01x03_Pin, J2 Conn_01x05_Pin, J3 Screw_Terminal_01x02, J5 Screw_Terminal_01x04, Q1 ME60N03, Q2 ME60N03

Commit message: use screw terminals from MF lib
Parts:
- J3: footprint TerminalBlock:TerminalBlock_bornier-2_P5.08mm -> MobiFlight:TerminalBlock_bornier-2_P5.08mm
- J5: footprint TerminalBlock:TerminalBlock_bornier-4_P5.08mm -> MobiFlight:TerminalBlock_bornier-4_P5.08mm
Changed lines of the file:
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@@
 			)
 		)
-		(property "Footprint" "TerminalBlock:TerminalBlock_bornier-2_P5.08mm"
+		(property "Footprint" "MobiFlight:TerminalBlock_bornier-2_P5.08mm"
 			(at 69.85 66.04 0)
 			(effects
@@
 			)
 		)
-		(property "Footprint" "TerminalBlock:TerminalBlock_bornier-4_P5.08mm"
+		(property "Footprint" "MobiFlight:TerminalBlock_bornier-4_P5.08mm"
 			(at 69.85 95.25 0)
 			(effects
