File: max7219-breakout-system/MAX7219-breakout-board.kicad_sch (KiCad schematic)
At the start: 22 parts, among them IC1 MAX7219CNG, IC2 MAX7219CNG, IC3 MAX7219CNG, IC4 MAX7219CNG, J1 Conn_01x05, J10 Conn_01x05, J2 Conn_02x08_Odd_Even, J3 Conn_02x08_Odd_Even, J4 Conn_02x08_Odd_Even, J5 Conn_02x08_Odd_Even, J6 Conn_02x08_Odd_Even, J7 Conn_02x08_Odd_Even, J8 Conn_02x08_Odd_Even, J9 Conn_02x08_Odd_Even

Commit message: changes for version 2.0
Parts:
- removed J1, J10: Conn_01x05, Connector_Molex:Molex_SPOX_5268-05A_1x05_P2.50mm_Horizontal, symbol Connector_Generic:Conn_01x05
- added C1, C3, C5, C7: 10µF, Capacitor_THT:CP_Radial_D5.0mm_P2.50mm, symbol Device:C_Polarized
- added J1: Conn_01x02_Male, Connector_JST:JST_XH_B2B-XH-A_1x02_P2.50mm_Vertical, symbol Connector:Conn_01x02_Male
- added J11, J2: Conn_01x05_Male, Connector_JST:JST_XH_B5B-XH-A_1x05_P2.50mm_Vertical, symbol Connector:Conn_01x05_Male
- added JP1: Jumper_3_Open, Connector_PinHeader_2.54mm:PinHeader_1x03_P2.54mm_Vertical, symbol Jumper:Jumper_3_Open
- renumbered C1 to C2, C2 to C4, C3 to C6, C4 to C8, J9 to J10, J2 to J3, J3 to J4, J4 to J5, J5 to J6, J6 to J7, J7 to J8, J8 to J9
Connections:
- net CLK: now also J11.4 (Pin_4), J2.4 (Pin_4); no longer IC1.12 (LOAD), IC1.18 (ISET), IC3.12 (LOAD), IC3.18 (ISET), IC4.12 (LOAD), IC4.18 (ISET), R1.2, R3.2, R4.2
- net DIG6-1: now also J3.14 (Pin_14)
- net DIG6-2: now also J5.14 (Pin_14)
- net DIG6-3: now also J7.14 (Pin_14)
- net DIG6-4: now also J9.14 (Pin_14)
- net DIG7-1: now also J3.16 (Pin_16)
- net DIG7-2: now also J5.16 (Pin_16)
- net DIG7-3: now also J7.16 (Pin_16)
- net DIG7-4: now also J9.16 (Pin_16)
- net DOUT4: now also J11.3 (Pin_3)
- net GND: now also C1.2, C3.2, C5.2, C7.2, J1.1 (Pin_1), J11.1 (Pin_1), J2.1 (Pin_1)
- net at IC2.18 (ISET), R2.2: no longer IC2.12 (LOAD)
- net +5V renamed VCC
- net VCC: now also C1.1, C3.1, C5.1, C7.1, J11.2 (Pin_2), JP1.2 (C)
- net DIN1 renamed DIN
- net DIN: now also J2.3 (Pin_3)
- new net: IC1.18 (ISET), R1.2
- new net: IC3.18 (ISET), R3.2
- new net: IC4.18 (ISET), R4.2
- new net: J1.2 (Pin_2), JP1.3 (B)
- new net: J2.2 (Pin_2), JP1.1 (A)
- new net LOAD(CS): IC1.12 (LOAD), IC2.12 (LOAD), IC3.12 (LOAD), IC4.12 (LOAD), J11.5 (Pin_5), J2.5 (Pin_5)
- no-connect marks 24 -> 16
Other:
- note added: "CLK"
- note added: "DIN"
- note added: "GND"
- note added: "JP1: 1-2 Power via MEGA-Module 2-3 Power via external Power"
- note added: "LOAD/CS"
- note added: "Vcc"

Commit message: mounting holes are 72mm apart (#28)
* mounting holes are 72mm apart
* Fixed all warnings, qr code, and jumper label
Parts:
- added H1, H2, H3, H4: MountingHole, MountingHole:MountingHole_3.2mm_M3_Pad, symbol Mechanical:MountingHole
- IC1, IC2, IC3, IC4: footprint Package_DIP:DIP-24_W7.62mm_MAX7219CNG -> Package_DIP:DIP-24_W7.62mm
- J10, J3, J4, J5, J6, J7, J8, J9: footprint Connector_IDC:IDC-Header_2x08_P2.54mm_Vertical -> mobiflight-library:IDC-Header_2x08_P2.54mm_Vertical
Connections:
- net CLK: now also J11.5 (Pin_5), J2.5 (Pin_5); no longer J11.4 (Pin_4), J2.4 (Pin_4)
- net 4 renamed SEG_F4
- net A1 renamed SEG_A1
- net A2 renamed SEG_A2
- net A3 renamed SEG_A3
- net A4 renamed SEG_A4
- net B1 renamed SEG_B1
- net B2 renamed SEG_B2
- net B3 renamed SEG_B3
- net B4 renamed SEG_B4
- net C1 renamed SEG_C1
- net C2 renamed SEG_C2
- net C3 renamed SEG_C3
- net C4 renamed SEG_C4
- net D1 renamed SEG_D1
- net D2 renamed SEG_D2
- net D3 renamed SEG_D3
- net D4 renamed SEG_D4
- net DIG0-1 renamed DIG0_1
- net DIG0-2 renamed DIG0_2
- net DIG0-3 renamed DIG0_3
- net DIG0-4 renamed DIG0_4
- net DIG1-1 renamed DIG1_1
- net DIG1-2 renamed DIG1_2
- net DIG1-3 renamed DIG1_3
- net DIG1-4 renamed DIG1_4
- net DIG2-1 renamed DIG2_1
- net DIG2-2 renamed DIG2_2
- net DIG2-3 renamed DIG2_3
- net DIG2-4 renamed DIG2_4
- net DIG3-1 renamed DIG3_1
- net DIG3-2 renamed DIG3_2
- net DIG3-3 renamed DIG3_3
- net DIG3-4 renamed DIG3_4
- net DIG4-1 renamed DIG4_1
- net DIG4-2 renamed DIG4_2
- net DIG4-3 renamed DIG4_3
- net DIG4-4 renamed DIG4_4
- net DIG5-1 renamed DIG5_1
- net DIG5-2 renamed DIG5_2
- net DIG5-3 renamed DIG5_3
- net DIG5-4 renamed DIG5_4
- net DIG6-1 renamed DIG6_1
- net DIG6-2 renamed DIG6_2
- net DIG6-3 renamed DIG6_3
- net DIG6-4 renamed DIG6_4
- net DIG7-1 renamed DIG7_1
- net DIG7-2 renamed DIG7_2
- net DIG7-3 renamed DIG7_3
- net DIG7-4 renamed DIG7_4
- net DP1 renamed SEG_DP1
- net DP2 renamed SEG_DP2
- net DP3 renamed SEG_DP3
- net DP4 renamed SEG_DP4
- net E1 renamed SEG_E1
- net E2 renamed SEG_E2
- net E3 renamed SEG_E3
- net E4 renamed SEG_E4
- net F1 renamed SEG_F1
- net F2 renamed SEG_F2
- net F3 renamed SEG_F3
- net G1 renamed SEG_G1
- net G2 renamed SEG_G2
- net G3 renamed SEG_G3
- net G4 renamed SEG_G4
- net LOAD(CS) renamed CS
- net CS: now also J11.4 (Pin_4), J2.4 (Pin_4); no longer J11.5 (Pin_5), J2.5 (Pin_5)
Other:
- note added: "DOUT"
- note added: "VCC"
- moved on the sheet: C3, C4, C7, IC2, IC3, IC4, J1, J10, J2, J3, J4, J5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

Commit message: fixed missing IDC footprints error
Parts:
- J10, J3, J4, J5, J6, J7, J8, J9: footprint mobiflight-library:IDC-Header_2x08_P2.54mm_Vertical -> MobiFlight:IDC-Header_2x08_P2.54mm_Vertical
Changed lines of the file:
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@@
 			)
 		)
-		(property "Footprint" "mobiflight-library:IDC-Header_2x08_P2.54mm_Vertical"
+		(property "Footprint" "MobiFlight:IDC-Header_2x08_P2.54mm_Vertical"
 			(at 109.22 142.24 0)
 			(effects
@@
 			)
 		)
-		(property "Footprint" "mobiflight-library:IDC-Header_2x08_P2.54mm_Vertical"
+		(property "Footprint" "MobiFlight:IDC-Header_2x08_P2.54mm_Vertical"
 			(at 109.22 172.085 0)
 			(effects
@@
 			)
 		)
-		(property "Footprint" "mobiflight-library:IDC-Header_2x08_P2.54mm_Vertical"
+		(property "Footprint" "MobiFlight:IDC-Header_2x08_P2.54mm_Vertical"
 			(at 224.79 144.78 0)
 			(effects
@@
 			)
 		)
-		(property "Footprint" "mobiflight-library:IDC-Header_2x08_P2.54mm_Vertical"
+		(property "Footprint" "MobiFlight:IDC-Header_2x08_P2.54mm_Vertical"
 			(at 224.79 171.45 0)
 			(effects
@@
 			)
 		)
-		(property "Footprint" "mobiflight-library:IDC-Header_2x08_P2.54mm_Vertical"
+		(property "Footprint" "MobiFlight:IDC-Header_2x08_P2.54mm_Vertical"
 			(at 358.775 145.415 0)
 			(effects
@@
 			)
 		)
-		(property "Footprint" "mobiflight-library:IDC-Header_2x08_P2.54mm_Vertical"
+		(property "Footprint" "MobiFlight:IDC-Header_2x08_P2.54mm_Vertical"
 			(at 358.775 172.085 0)
 			(effects
@@
 			)
 		)
-		(property "Footprint" "mobiflight-library:IDC-Header_2x08_P2.54mm_Vertical"
+		(property "Footprint" "MobiFlight:IDC-Header_2x08_P2.54mm_Vertical"
 			(at 495.3 144.78 0)
 			(effects
@@
 			)
 		)
-		(property "Footprint" "mobiflight-library:IDC-Header_2x08_P2.54mm_Vertical"
+		(property "Footprint" "MobiFlight:IDC-Header_2x08_P2.54mm_Vertical"
 			(at 495.3 171.45 0)
 			(effects

Commit message: use MAX7219 symbol from MF lib
Parts:
- IC1, IC2, IC3, IC4: symbol MAX7219CNG:MAX7219CNG -> mobiflight-library:MAX7219CNG
Changed lines of the file:
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@@
 	)
 	(symbol
-		(lib_id "MAX7219CNG:MAX7219CNG")
+		(lib_id "mobiflight-library:MAX7219CNG")
 		(at 107.315 83.82 270)
 		(unit 1)
@@
 	)
 	(symbol
-		(lib_id "MAX7219CNG:MAX7219CNG")
+		(lib_id "mobiflight-library:MAX7219CNG")
 		(at 223.52 90.17 270)
 		(unit 1)
@@
 	)
 	(symbol
-		(lib_id "MAX7219CNG:MAX7219CNG")
+		(lib_id "mobiflight-library:MAX7219CNG")
 		(at 356.235 90.17 270)
 		(unit 1)
@@
 	)
 	(symbol
-		(lib_id "MAX7219CNG:MAX7219CNG")
+		(lib_id "mobiflight-library:MAX7219CNG")
 		(at 490.855 90.17 270)
 		(unit 1)
