File: dual-encoder-board/dual-encoder-board.kicad_pcb (KiCad board)
At the start: 2 copper layers, 27.3 x 27.3 mm, 8 parts, among them U1 EC11EBB24C03

Commit message: use footprint and symbol for Dual Encoder from MF lib
Parts:
- U1: footprint MobiFlight:EC11EBB24C03 -> MobiFlight:EC11EBB24C03_oval
Other:
- board text removed: "JLCJLCJLCJLC"
Changed lines of the file:
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@@
 			)
 		)
-		(property "Datasheet" ""
+		(property "Datasheet" "~"
 			(at 0 0 180)
 			(layer "F.Fab")
@@
 			)
 		)
-		(property "Description" "Mounting Hole with connection"
+		(property "Description" ""
 			(at 0 0 180)
 			(layer "F.Fab")
@@
 			)
 		)
+		(property ki_fp_filters "MountingHole*Pad*")
+		(sheetname "/")
 		(sheetfile "dual-encoder-board.kicad_sch")
 		(attr exclude_from_pos_files)
@@
 			)
 		)
-		(property "Datasheet" ""
+		(property "Datasheet" "~"
 			(at 0 0 180)
 			(layer "F.Fab")
@@
 			)
 		)
-		(property "Description" "Mounting Hole with connection"
+		(property "Description" ""
 			(at 0 0 180)
 			(layer "F.Fab")
@@
 			)
 		)
+		(property ki_fp_filters "MountingHole*Pad*")
+		(sheetname "/")
 		(sheetfile "dual-encoder-board.kicad_sch")
 		(attr exclude_from_pos_files)
@@
 			)
 		)
-		(property "Datasheet" ""
+		(property "Datasheet" "~"
 			(at 0 0 180)
 			(layer "F.Fab")
@@
 			)
 		)
-		(property "Description" "Mounting Hole with connection"
+		(property "Description" ""
 			(at 0 0 180)
 			(layer "F.Fab")
@@
 			)
 		)
+		(property ki_fp_filters "MountingHole*Pad*")
+		(sheetname "/")
 		(sheetfile "dual-encoder-board.kicad_sch")
 		(attr exclude_from_pos_files)
@@
 			)
 		)
-		(property "Datasheet" ""
+		(property "Datasheet" "~"
 			(at 0 0 180)
 			(layer "F.Fab")
@@
 			)
 		)
-		(property "Description" "Mounting Hole with connection"
+		(property "Description" ""
 			(at 0 0 180)
 			(layer "F.Fab")
@@
 			)
 		)
+		(property ki_fp_filters "MountingHole*Pad*")
+		(sheetname "/")
 		(sheetfile "dual-encoder-board.kicad_sch")
 		(attr exclude_from_pos_files)
@@
 		(embedded_fonts no)
 	)
-	(footprint "MobiFlight:EC11EBB24C03"
+	(footprint "MobiFlight:EC11EBB24C03_oval"
 		(layer "F.Cu")
 		(at 117.994914 66.070016 180)
@@
 			)
 		)
-		(property "Datasheet" ""
+		(property "Datasheet" "https://componentsearchengine.com/Datasheets/2/EC11EBB24C03.pdf"
 			(at 0 0 180)
 			(layer "F.Fab")
@@
 			)
 		)
+		(sheetname "/")
 		(sheetfile "dual-encoder-board.kicad_sch")
 		(attr through_hole)
@@
 			)
 		)
-		(property "Datasheet" ""
+		(property "Datasheet" "~"
 			(at 0 0 90)
 			(layer "F.Fab")
@@
 			)
 		)
-		(property "Description" "Generic connector, single row, 01x04, script generated (kicad-library-utils/schlib/autogen/connector/)"
+		(property "Description" ""
 			(at 0 0 90)
 			(layer "F.Fab")
@@
 			)
 		)
+		(property ki_fp_filters "Connector*:*_1x??_*")
+		(sheetname "/")
 		(sheetfile "dual-encoder-board.kicad_sch")
 		(attr through_hole)
@@
 			)
 		)
-		(property "Datasheet" ""
+		(property "Datasheet" "~"
 			(at 0 0 270)
 			(layer "F.Fab")
@@
 			)
 		)
-		(property "Description" "Generic connector, single row, 01x04, script generated (kicad-library-utils/schlib/autogen/connector/)"
+		(property "Description" ""
 			(at 0 0 270)
 			(layer "F.Fab")
@@
 			)
 		)
+		(property ki_fp_filters "Connector*:*_1x??_*")
+		(sheetname "/")
 		(sheetfile "dual-encoder-board.kicad_sch")
 		(attr through_hole)
@@
 		)
 	)
-	(gr_text "JLCJLCJLCJLC"
-		(at 117.994914 78.770016 0)
-		(layer "B.SilkS")
-		(effects
-			(font
-				(size 0.8 0.8)
-				(thickness 0.15)
-			)
-			(justify mirror)
-		)
-	)
