File: max7219-breakout-digits/7-Segment_V5_3er.kicad_pcb (KiCad board)
At the start: 2 copper layers, 47.8 x 10.7 mm, 5 parts, among them J1 Conn_02x08_Odd_Even, U1 7Segment 3 digit common catho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

Commit message: labeling with # digits and not 2.8mm
Other:
- board text added: "MobiFlight Display System 3 Digits ${REVISION}"
- board text removed: "MobiFlight Display System 2.8mm ${REVISION}"
Changed lines of the file:
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@@
 		(layer "Edge.Cuts")
 	)
-	(gr_text "MobiFlight\nDisplay\nSystem\n2.8mm\n${REVISION}"
-		(at 121.158 60.96 0)
+	(gr_text "MobiFlight Display System 3 Digits ${REVISION}"
+		(at 116.16 59.38 0)
 		(layer "B.SilkS")
 		(effects
 			(font
 				(size 0.5 0.5)
-				(thickness 0.125)
+				(thickness 0.15)
 			)
-			(justify mirror)
+			(justify left bottom mirror)
 		)
 	)
