File: max7219-breakout-digits/7-Segment_V5_4er.kicad_pcb (KiCad board)
At the start: 2 copper layers, 51 x 12 mm, 5 parts, among them J1 Conn_02x08_Odd_Even, U1 HDSM-443B_CC_2Digit_7Segment_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, U2 HDSM-443B_CC_2Digit_7Segment_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

Commit message: labeling with # digits and not 2.8mm
Other:
- board text added: "MobiFlight Display System 4 Digits ${REVISION}"
- board text removed: "MobiFlight Display System 2.8mm ${REVISION}"
Changed lines of the file:
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@@
 		(layer "Edge.Cuts")
 	)
-	(gr_text "MobiFlight Display System 2.8mm ${REVISION}"
+	(gr_text "MobiFlight Display System 4 Digits ${REVISION}"
 		(at 95.606511 54.42064 0)
 		(layer "B.SilkS")
