File: max7219-breakout-digits/7-Segment_V5_6er.kicad_pcb (KiCad board)
At the start: 2 copper layers, 66 x 12 mm, 6 parts, among them J1 Conn_02x08_Odd_Even, U1 7Segment 3 digit CC_STH, U2 7Segment 3 digit CC_STH

Commit message: labeling with # digits and not 2.8mm
Other:
- board text added: "MobiFlight Display System 6 Digits ${REVISION}"
- board text removed: "MobiFlight Display System 2.8mm ${REVISION}"
Changed lines of the file:
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@@
 		(layer "Edge.Cuts")
 	)
-	(gr_text "MobiFlight Display System 2.8mm ${REVISION}"
+	(gr_text "MobiFlight Display System 6 Digits ${REVISION}"
 		(at 91.4566 57.5553 0)
 		(layer "B.SilkS")
