File: max7219-breakout-digits/3-digits_0.28.kicad_sch (KiCad schematic)
At the start: 4 parts, among them J1 Conn_02x08_Odd_Even, U1 7Segment 3 digit common catho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

Commit message: add .35 symbols and footprints, rework 3 and 4 digit 0.35
Other:
- title: 7 Segment Display Module, 3 digits -> 7-Segment Display Module, 3 Digits
Changed lines of the file:
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@@
 	(paper "A5")
 	(title_block
-		(title "7 Segment Display Module, 3 digits")
+		(title "7-Segment Display Module, 3 Digits")
 		(date "2025-12")
 		(rev "V6.0")

Commit message: rotate IDC on 0.28 displays, plated mounting holes for 0.35 displays, set version for 0.35 displays
Other:
- title: 7-Segment Display Module, 3 Digits -> 7-Segment Display Module 0.28, 3 Digits
Changed lines of the file:
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@@
 	(paper "A5")
 	(title_block
-		(title "7-Segment Display Module, 3 Digits")
+		(title "7-Segment Display Module 0.28, 3 Digits")
 		(date "2025-12")
-		(rev "V6.0")
+		(rev "V5.2")
 		(company "MobiFlight")
 	)
