File: max7219-breakout-digits/3-digits_0.36.kicad_sch (KiCad schematic)
At the start: 4 parts, among them J1 Conn_02x08_Odd_Even, U1 HDSM-443B_7-Segment_3_Digit

Commit message: rename everything from 0.35 to 0.36
Parts:
- U1: footprint MobiFlight:STH_7_3 Digits_0.35_CC -> MobiFlight:STH_7_3 Digits_0.36_CC; symbol MobiFlight:7Segment 3 digit 0.35 common cathode STH -> MobiFlight:7Segment 3 digit 0.36 common cathode STH
Other:
- title: 7-Segment Display Module 0.35, 3 Digits -> 7-Segment Display Module 0.36, 3 Digits
Changed lines of the file:
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@@
 	(paper "A5")
 	(title_block
-		(title "7-Segment Display Module 0.35, 3 Digits")
+		(title "7-Segment Display Module 0.36, 3 Digits")
 		(date "2025-12")
 		(rev "V5.1")
@@
 	)
 	(symbol
-		(lib_id "MobiFlight:7Segment 3 digit 0.35 common cathode STH")
+		(lib_id "MobiFlight:7Segment 3 digit 0.36 common cathode STH")
 		(at 71.628 44.704 0)
 		(unit 1)
@@
 			)
 		)
-		(property "Footprint" "MobiFlight:STH_7_3 Digits_0.35_CC"
+		(property "Footprint" "MobiFlight:STH_7_3 Digits_0.36_CC"
 			(at 75.184 64.008 0)
 			(effects
