File: max7219SMD-breakout-system/max7219SMD-breakout-system.kicad_sch (KiCad schematic)
At the start: 32 parts, among them IC1 MAX7219CNG, IC2 MAX7219CNG, IC3 MAX7219CNG, IC4 MAX7219CNG, J1 Conn_01x02_Male, J10 Conn_02x08_Odd_Even, J11 Conn_01x05_Male, J2 Conn_01x05_Male, J3 Conn_02x08_Odd_Even, J4 Conn_02x08_Odd_Even, J5 Conn_02x08_Odd_Even, J6 Conn_02x08_Odd_Even, J7 Conn_02x08_Odd_Even, J8 Conn_02x08_Odd_Even, J9 Conn_02x08_Odd_Even

Commit message: everything routed
Parts:
- removed JP1: Jumper_3_Open, Connector_PinHeader_2.54mm:PinHeader_1x03_P2.54mm_Vertical, symbol Jumper:Jumper_3_Open
- added D1, D2: D_Schottky_B5819W-SL, Diode_SMD:D_SOD-123, symbol MobiFlight:D_Schottky_B5819W-SL
- C1, C3, C5, C7: value 10µF -> 47uF; footprint Capacitor_THT:CP_Radial_D5.0mm_P2.50mm -> Capacitor_Tantalum_SMD:CP_EIA-3528-21_Kemet-B; symbol Device:C_Polarized -> MobiFlight:C_Polarized_Tantal_47u; LCSC (none) -> C123253
- C2, C4, C6, C8: value 0,1µF -> 100nF; footprint Capacitor_THT:C_Disc_D5.0mm_W2.5mm_P5.00mm -> Capacitor_SMD:C_0805_2012Metric
- H1, H2, H3, H4: now left out of the parts list
- IC1, IC2, IC3, IC4: footprint Package_DIP:DIP-24_W7.62mm -> Package_SO:SOIC-24W_7.5x15.4mm_P1.27mm; symbol mobiflight-library:MAX7219CNG -> MobiFlight:MAX7219_SMD; LCSC (none) -> C5145464
- R1, R2, R3, R4: footprint Resistor_THT:R_Axial_DIN0204_L3.6mm_D1.6mm_P7.62mm_Horizontal -> Resistor_SMD:R_0805_2012Metric
Connections:
- net VCC: now also D2.1 (K)
- net at J1.2 (Pin_2): now also D1.1 (K), D2.2 (A)
- net at J2.2 (Pin_2): now also D1.2 (A)
Other:
- note added: "Vboard"
- note added: "Vextern"
- note removed: "JP1: 1-2 Power via MEGA-Module 2-3 Power via external Power"
- note removed: "Vcc"
- title: MAX7219  -> MAX7219 SMD Breakout Board
- moved on the sheet: C1, C2, C3, C4, C5, C6, C7, C8, H1, H2, H3, H4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

Commit message: PCB optimazations
Parts:
- J1: symbol Connector:Conn_01x02_Male -> MobiFlight:JST-XH_02_Pin_vertical_red; LCSC (none) -> C24192
- J10, J3, J4, J5, J6, J7, J8, J9: symbol Connector_Generic:Conn_02x08_Odd_Even -> MobiFlight:IDC_conn_02x08; LCSC (none) -> C3406
- J11, J2: symbol Connector:Conn_01x05_Male -> MobiFlight:JST-XH_05_Pin_vertical; LCSC (none) -> C2318
Changed lines of the file:
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@@
 	(text "Vboard"
 		(exclude_from_sim no)
-		(at 37.084 59.182 0)
+		(at 33.782 59.436 0)
 		(effects
 			(font
@@
 	(text "Vextern"
 		(exclude_from_sim no)
-		(at 36.83 41.91 0)
+		(at 34.036 41.91 0)
 		(effects
 			(font
@@
 	)
 	(symbol
-		(lib_id "Connector_Generic:Conn_02x08_Odd_Even")
+		(lib_id "MobiFlight:IDC_conn_02x08")
 		(at 76.2 194.31 0)
 		(unit 1)
@@
 			)
 		)
-		(property "Description" ""
+		(property "Description" "Generic connector, double row, 02x08, odd/even pin numbering scheme (row 1 odd numbers, row 2 even numbers), script generated (kicad-library-utils/schlib/autogen/connector/)"
 			(at 76.2 194.31 0)
 			(effects
@@
 					(size 1.27 1.27)
 				)
+				(hide yes)
+			)
+		)
+		(property "LCSC" "C3406"
+			(at 76.2 194.31 0)
+			(effects
+				(font
+					(size 1.27 1.27)
+				)
+				(hide yes)
 			)
 		)
@@
 	)
 	(symbol
-		(lib_id "Connector_Generic:Conn_02x08_Odd_Even")
+		(lib_id "MobiFlight:IDC_conn_02x08")
 		(at 76.2 224.79 0)
 		(unit 1)
@@
 			)
 		)
-		(property "Description" ""
+		(property "Description" "Generic connector, double row, 02x08, odd/even pin numbering scheme (row 1 odd numbers, row 2 even numbers), script generated (kicad-library-utils/schlib/autogen/connector/)"
+			(at 76.2 224.79 0)
+			(effects
+				(font
+					(size 1.27 1.27)
+				)
+				(hide yes)
+			)
+		)
+		(property "LCSC" "C3406"
 			(at 76.2 224.79 0)
 			(effects
@@
 					(size 1.27 1.27)
 				)
+				(hide yes)
 			)
 		)
@@
 	)
 	(symbol
-		(lib_id "Connector_Generic:Conn_02x08_Odd_Even")
+		(lib_id "MobiFlight:IDC_conn_02x08")
 		(at 161.29 196.85 0)
 		(unit 1)
@@
 			)
 		)
-		(property "Description" ""
+		(property "Description" "Generic connector, double row, 02x08, odd/even pin numbering scheme (row 1 odd numbers, row 2 even numbers), script generated (kicad-library-utils/schlib/autogen/connector/)"
+			(at 161.29 196.85 0)
+			(effects
+				(font
+					(size 1.27 1.27)
+				)
+				(hide yes)
+			)
+		)
+		(property "LCSC" "C3406"
 			(at 161.29 196.85 0)
 			(effects
@@
 					(size 1.27 1.27)
 				)
+				(hide yes)
 			)
 		)
@@
 	)
 	(symbol
-		(lib_id "Connector_Generic:Conn_02x08_Odd_Even")
+		(lib_id "MobiFlight:IDC_conn_02x08")
 		(at 161.29 223.52 0)
 		(unit 1)
@@
 			)
 		)
-		(property "Description" ""
+		(property "Description" "Generic connector, double row, 02x08, odd/even pin numbering scheme (row 1 odd numbers, row 2 even numbers), script generated (kicad-library-utils/schlib/autogen/connector/)"
+			(at 161.29 223.52 0)
+			(effects
+				(font
+					(size 1.27 1.27)
+				)
+				(hide yes)
+			)
+		)
+		(property "LCSC" "C3406"
 			(at 161.29 223.52 0)
 			(effects
@@
 					(size 1.27 1.27)
 				)
+				(hide yes)
 			)
 		)
@@
 	)
 	(symbol
-		(lib_id "Connector_Generic:Conn_02x08_Odd_Even")
+		(lib_id "MobiFlight:IDC_conn_02x08")
 		(at 260.35 198.12 0)
 		(unit 1)
@@
 			)
 		)
-		(property "Description" ""
+		(property "Description" "Generic connector, double row, 02x08, odd/even pin numbering scheme (row 1 odd numbers, row 2 even numbers), script generated (kicad-library-utils/schlib/autogen/connector/)"
 			(at 260.35 198.12 0)
 			(effects
@@
 					(size 1.27 1.27)
 				)
+				(hide yes)
+			)
+		)
+		(property "LCSC" "C3406"
+			(at 260.35 198.12 0)
+			(effects
+				(font
+					(size 1.27 1.27)
+				)
+				(hide yes)
 			)
 		)
@@
 	)
 	(symbol
-		(lib_id "Connector_Generic:Conn_02x08_Odd_Even")
+		(lib_id "MobiFlight:IDC_conn_02x08")
 		(at 260.35 224.79 0)
 		(unit 1)
@@
 			)
 		)
-		(property "Description" ""
+		(property "Description" "Generic connector, double row, 02x08, odd/even pin numbering scheme (row 1 odd numbers, row 2 even numbers), script generated (kicad-library-utils/schlib/autogen/connector/)"
+			(at 260.35 224.79 0)
+			(effects
+				(font
+					(size 1.27 1.27)
+				)
+				(hide yes)
+			)
+		)
+		(property "LCSC" "C3406"
 			(at 260.35 224.79 0)
 			(effects
@@
 					(size 1.27 1.27)
 				)
+				(hide yes)
 			)
 		)
@@
 	)
 	(symbol
-		(lib_id "Connector_Generic:Conn_02x08_Odd_Even")
+		(lib_id "MobiFlight:IDC_conn_02x08")
 		(at 355.6 199.39 0)
 		(unit 1)
@@
 			)
 		)
-		(property "Description" ""
+		(property "Description" "Generic connector, double row, 02x08, odd/even pin numbering scheme (row 1 odd numbers, row 2 even numbers), script generated (kicad-library-utils/schlib/autogen/connector/)"
+			(at 355.6 199.39 0)
+			(effects
+				(font
+					(size 1.27 1.27)
+				)
+				(hide yes)
+			)
+		)
+		(property "LCSC" "C3406"
 			(at 355.6 199.39 0)
 			(effects
@@
 					(size 1.27 1.27)
 				)
+				(hide yes)
 			)
 		)
@@
 	)
 	(symbol
-		(lib_id "Connector_Generic:Conn_02x08_Odd_Even")
+		(lib_id "MobiFlight:IDC_conn_02x08")
 		(at 355.6 226.06 0)
 		(unit 1)
@@
 			)
 		)
-		(property "Description" ""
+		(property "Description" "Generic connector, double row, 02x08, odd/even pin numbering scheme (row 1 odd numbers, row 2 even numbers), script generated (kicad-library-utils/schlib/autogen/connector/)"
+			(at 355.6 226.06 0)
+			(effects
+				(font
+					(size 1.27 1.27)
+				)
+				(hide yes)
+			)
+		)
+		(property "LCSC" "C3406"
 			(at 355.6 226.06 0)
 			(effects
@@
 					(size 1.27 1.27)
 				)
+				(hide yes)
 			)
 		)
@@
 	)
 	(symbol
-		(lib_id "Connector:Conn_01x02_Male")
+		(lib_id "MobiFlight:JST-XH_02_Pin_vertical_red")
 		(at 41.91 38.1 0)
 		(unit 1)
@@
 		)
 		(property "Value" "Conn_01x02_Male"
-			(at 39.624 30.988 0)
+			(at 26.924 39.37 0)
 			(effects
 				(font
@@
 			)
 		)
-		(property "Description" ""
+		(property "Description" "Generic connector, single row, 01x02, script generated"
 			(at 41.91 38.1 0)
 			(effects
@@
 					(size 1.27 1.27)
 				)
+				(hide yes)
+			)
+		)
+		(property "LCSC" "C24192"
+			(at 47.244 42.926 0)
+			(effects
+				(font
+					(size 1.27 1.27)
+				)
 			)
 		)
@@
 	)
 	(symbol
-		(lib_id "Connector:Conn_01x05_Male")
+		(lib_id "MobiFlight:JST-XH_05_Pin_vertical")
 		(at 160.02 44.45 0)
 		(mirror y)
@@
 			)
 		)
-		(property "Description" ""
+		(property "Description" "Generic connector, single row, 01x05, script generated"
 			(at 160.02 44.45 0)
 			(effects
@@
 					(size 1.27 1.27)
 				)
+				(hide yes)
+			)
+		)
+		(property "LCSC" "C2318"
+			(at 158.496 52.578 0)
+			(effects
+				(font
+					(size 1.27 1.27)
+				)
 			)
 		)
@@
 	)
 	(symbol
-		(lib_id "Connector:Conn_01x05_Male")
+		(lib_id "MobiFlight:JST-XH_05_Pin_vertical")
 		(at 41.91 60.96 0)
 		(unit 1)
@@
 		)
 		(property "Value" "Conn_01x05_Male"
-			(at 28.194 52.578 0)
+			(at 25.654 59.944 0)
 			(effects
 				(font
@@
 			)
 		)
-		(property "Description" ""
+		(property "Description" "Generic connector, single row, 01x05, script generated"
 			(at 41.91 60.96 0)
 			(effects
 				(font
+					(size 1.27 1.27)
+				)
+				(hide yes)
+			)
+		)
+		(property "LCSC" "C2318"
+			(at 43.688 68.834 0)
+			(effects
+				(font
