File: toggle-switch-board/toggle-switch-board.kicad_sch (KiCad schematic)
At the start: 6 parts, among them J1 JST-XH_03_Pin_vertical, SW1 SW_SPST

Commit message: fix symbol property to match the actual symbol type
this was a leftover from changing symbols, good catch.

Co-authored-by: Copilot Autofix powered by AI <175728472+Copilot@users.noreply.github.com>
Parts:
- SW1: value SW_SPST -> SW_SPDT
Changed lines of the file:
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@@
 			)
 		)
-		(property "Value" "SW_SPST"
+		(property "Value" "SW_SPDT"
 			(at 49.53 69.85 0)
 			(show_name no)
