File: piconano/piconano.kicad_sch (KiCad schematic)
At the start: 3 parts, among them SW1 SW_Push, SW2 SW_Push

Commit message: update revision and date
Other:
- title: RP2350A Template -> PicoNano
Changed lines of the file:
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@@
 	(paper "A4")
 	(title_block
-		(title "RP2350A Template")
-		(date "2025-10-10")
-		(rev "REV0")
+		(title "PicoNano")
+		(date "2026-07")
+		(rev "1.0.0")
 		(company "MobiFlight")
 	)
@@
 		(property "Description" "Push button switch, generic, two pins"
 			(at 201.93 134.62 0)
+			(hide yes)
 			(show_name no)
 			(do_not_autoplace no)
@@
 		(property "Description" "Push button switch, generic, two pins"
 			(at 157.48 134.62 0)
-			(show_name no)
-			(do_not_autoplace no)
+			(hide yes)
+			(show_name no)
+			(do_not_autoplace no)
