File: picomega/picomega.kicad_sch (KiCad schematic)
At the start: 27 parts, among them J5 PicoMega, Q4 BSS138, Q5 BSS138, Q6 BSS138, Q7 BSS138, SW1 SW_Push, U4 AMS1117-5.0 SOT-223

Commit message: without level shifter
Parts:
- removed JP2: SolderJumper_3_Open, MobiFlight:SolderJumper-3_P1.3mm_Open_RoundedPad1.0x1.5mm, symbol MobiFlight:SolderJumper_3_Open
- removed Q4, Q5, Q6, Q7: BSS138, Package_TO_SOT_SMD:SOT-23, symbol Transistor_FET:BSS138
- removed R16, R17, R18, R19, R20, R21, R23, R24: 10k, Resistor_SMD:R_0402_1005Metric, symbol Device:R
- J5: footprint Own_Library:PicoMega -> MobiFlight:PicoMega
Connections:
- net GPIO22_LS is gone; now on net GND: J5.33 (GND)
- net GPIO23_LS is gone; now on net GND: J5.34 (GND)
- net GPIO24_LS is gone; now on net GND: J5.35 (GND)
- net GPIO25_LS is gone; now on net GND: J5.36 (GND)
- net GND: no longer J5.31 (GND), J5.32 (GND), J5.37 (GND), J5.38 (GND)
- net GPIO22: now also J5.31 (D22)
- net GPIO23: now also J5.32 (D23)
- net GPIO24: now also J5.37 (D24)
- net GPIO25: now also J5.38 (D25)
Other:
- note removed: "Level Shifter"
- moved on the sheet: C19, C22, C23, C24, C25, C26, D2, SW1, U4

Commit message: update for JLCPCB BOM
Parts:
- J5: now left out of the parts list
Changed lines of the file:
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@@
 		(body_style 1)
 		(exclude_from_sim no)
-		(in_bom yes)
+		(in_bom no)
 		(on_board yes)
 		(in_pos_files yes)

Commit message: moved over to RP23545B
Other:
- sheet RP2350B renamed RP2354B
- sheet RP2354B: file RP2350B.kicad_sch -> RP2354B.kicad_sch
Changed lines of the file:
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@@
 			(color 0 0 0 0)
 		)
-		(property "Sheetname" "RP2350B"
+		(property "Sheetname" "RP2354B"
 			(at 39.37 53.8984 0)
 			(show_name no)
@@
 			)
 		)
-		(property "Sheetfile" "RP2350B.kicad_sch"
+		(property "Sheetfile" "RP2354B.kicad_sch"
 			(at 39.37 208.8646 0)
 			(show_name no)

Commit message: add Reset Button for PicoMega
Parts:
- added SW2: SW_Push, Own_Library:SW_Push_1P1T_NO_Vertical_Wuerth_434133025816, symbol MobiFlight:Switch_SMD_5x5_Wuerth
Connections:
- net GND: now also SW2.1
- new net RESET: SW2.2
- no-connect marks 1 -> 0
Other:
- note added: "Reset"
