File: picomega/RP2354B.kicad_sch (KiCad schematic)
At the start: 35 parts, among them J1 USB_C_Receptacle_USB2.0_16P, U1 RP2350_80QFN, U2 AMS1117-3.3 SOT-223, Y1 ABM8-272-T3

Commit message: update USB connector in library and for PicoMega
Parts:
- J1: JLCPCB C2997432 -> C393939; LCSC C2997432 -> (none)
Changed lines of the file:
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@@
 			)
 		)
-		(property "JLCPCB" "C2997432"
+		(property "JLCPCB" "C393939"
 			(at 45.72 193.04 0)
 			(show_name no)
 			(do_not_autoplace no)
-			(effects
-				(font
-					(size 1.27 1.27)
-				)
-			)
-		)
-		(property "LCSC" "C2997432"
-			(at 45.72 195.58 0)
-			(hide yes)
-			(show_name no)
-			(do_not_autoplace no)
-			(effects
-				(font
-					(size 1.27 1.27)
-				)
-			)
-		)
-		(property "SLC" ""
-			(at 45.72 215.9 0)
-			(hide yes)
-			(show_name no)
-			(do_not_autoplace no)

Commit message: add Reset Button for PicoMega
Parts:
- C20: value 4.7uF -> 4.7u
Changed lines of the file:
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@@
 			)
 		)
-		(property "Value" "4.7uF"
+		(property "Value" "4.7u"
 			(at 298.831 63.373 0)
 			(show_name no)

Commit message: update symbols for RP2354A/B
Parts:
- U1: value RP2350_80QFN -> RP2354_80QFN; LCSC C39843328 -> (none)
Other:
- note added: "Make sure R7 and R8 are close to RP2354B"
- note removed: "Make sure R7 and R8 are close to RP2350A"
Changed lines of the file:
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@@
 		)
 	)
-	(text "Make sure R7 and R8 are\nclose to RP2350A"
+	(text "Make sure R7 and R8 are\nclose to RP2354B"
 		(exclude_from_sim no)
 		(at 320.802 81.026 0)
@@
 			)
 		)
-		(property "Value" "RP2350_80QFN"
+		(property "Value" "RP2354_80QFN"
 			(at 268.8433 222.25 0)
 			(show_name no)
@@
 			)
 		)
-		(property "LCSC" "C39843328"
-			(at 268.8433 227.33 0)
-			(hide yes)
-			(show_name no)
-			(do_not_autoplace no)
-			(effects
-				(font
-					(size 1.27 1.27)
-				)
-				(justify left)
-			)
-		)
-		(property "SLC" ""
-			(at 266.7 142.24 0)
-			(hide yes)
-			(show_name no)
-			(do_not_autoplace no)
-			(effects
-				(font
-					(size 1.27 1.27)
-				)
-			)
-		)
